File: ps-ohk/ps-ohk.kicad_sch (KiCad schematic)
At the start: 26 parts

Commit message: Added 40-pin IO Expander to project
Will make use of two of them

Signed-off-by: Dylan Turner <dylan.turner@tutanota.com>
Parts:
- added IC_IOEXP1: PCA9505DGGY, PCA9505DGGY:SOP50P810X120-56N, symbol PCA9505DGGY:PCA9505DGGY
Connections:
- net KEY_A: now also IC_IOEXP1.3 (IO0_0)
