File: keys-righthand/keys-righthand.kicad_pcb (KiCad board)
At the start: 2 copper layers, 190.6 x 229.6 mm, 83 parts, among them J1 Conn_01x20, J2 Conn_01x20, J3 Conn_01x20, J4 Conn_01x20

Commit message: keys-righthand: wired up
Signed-off-by: Dylan Turner <dylan.turner@tutanota.com>
Parts:
- moved J1 203.9 mm to (22.6, 159.6)
- moved J2 203.9 mm to (50.1, 135.5)
- moved J3 203.9 mm to (50.1, 111.3)
- moved J4 203.9 mm to (41.6, 103.7)
- moved S_1 170.9 mm to (198.1, 96.5)
- moved S_CAPS1 170.9 mm to (198.1, 137.2)
- moved S_COMMA1 170.9 mm to (198.1, 76.2)
- moved S_GRAVE1 170.9 mm to (198.1, 116.8)
- moved S_LBK1 170.9 mm to (198.1, 35.6)
- moved S_SEMI1 170.9 mm to (198.1, 55.9)
- moved S_SHIFT1 170.9 mm to (198.1, 177.8)
- moved S_TAB1 170.9 mm to (198.1, 157.5)
- moved S_F12 170.9 mm to (27.9, 45.7)
- moved S_F6 170.9 mm to (27.9, 25.4)
- moved S_PGU1 155.7 mm to (35.6, 66.0)
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Routing:
- net GND: track 0.00 -> 1878.1 mm, vias 0 -> 36
- net /KEY_Q: track 0.00 -> 512.2 mm, vias 0 -> 8
- net /KEY_EQ: track 0.00 -> 480.6 mm, vias 0 -> 6
- net /KEY_DASH: track 0.00 -> 422.7 mm, vias 0 -> 5
- net /KEY_RET: track 0.00 -> 387.7 mm, vias 0 -> 5
- net /KEY_U: track 0.00 -> 383.1 mm, vias 0 -> 5
- net /KEY_F6: track 0.00 -> 265.9 mm, vias 0 -> 5
- net /KEY_LBK: track 0.00 -> 258.5 mm, vias 0 -> 5
- net /KEY_ESC: track 0.00 -> 255.8 mm, vias 0 -> 7
- net /KEY_F1: track 0.00 -> 243.1 mm, vias 0 -> 6
- net /KEY_RBK: track 0.00 -> 240.0 mm, vias 0 -> 5
- net /KEY_SEMI: track 0.00 -> 238.7 mm, vias 0 -> 5
- net /KEY_CTRL: track 0.00 -> 231.6 mm, vias 0 -> 7
- net /KEY_F7: track 0.00 -> 230.6 mm, vias 0 -> 3
- net /KEY_F4: track 0.00 -> 229.7 mm, vias 0 -> 8
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
Commit message: pcb: Update revision numbers
Signed-off-by: Dylan Turner <dylan.turner@tutanota.com>
Other:
- board text added: "r3"
- board text removed: "r2"
Changed lines of the file:
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@@
 	(title_block
 		(title "PS-OHK")
-		(date "2024-06-18")
-		(rev "2")
+		(date "2024-06-25")
+		(rev "3")
 		(company "Polymath-Studio")
 	)
@@
 		)
 	)
-	(gr_text "r2"
+	(gr_text "r3"
 		(at 155.4734 58.166 0)
 		(layer "B.SilkS")
