File: keys-righthand/keys-righthand.kicad_sch (KiCad schematic)
At the start: 4 parts, among them J1 Conn_01x20, J2 Conn_01x20, J3 Conn_01x20, J4 Conn_01x20

Commit message: pcb: Update revision numbers
Signed-off-by: Dylan Turner <dylan.turner@tutanota.com>
Other:
- title: PS-OHK Keys (Left-Hand) -> PS-OHK Keys (Right-Hand)
Changed lines of the file:
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@@
 	(paper "A4")
 	(title_block
-		(title "PS-OHK Keys (Left-Hand)")
-		(date "2024-06-24")
-		(rev "2")
+		(title "PS-OHK Keys (Right-Hand)")
+		(date "2024-06-25")
+		(rev "3")
 		(company "Polymath-Studio")
 	)
@@
 		)
 		(instances
-			(project "keys-lefthand"
+			(project "keys-righthand"
 				(path "/9764b4ba-7c88-49a9-89e6-e6f35382ac72"
 					(reference "J4")
@@
 		)
 		(instances
-			(project "keys-lefthand"
+			(project "keys-righthand"
 				(path "/9764b4ba-7c88-49a9-89e6-e6f35382ac72"
 					(reference "J1")
@@
 		)
 		(instances
-			(project "keys-lefthand"
+			(project "keys-righthand"
 				(path "/9764b4ba-7c88-49a9-89e6-e6f35382ac72"
 					(reference "#PWR0112")
@@
 		)
 		(instances
-			(project "keys-lefthand"
+			(project "keys-righthand"
 				(path "/9764b4ba-7c88-49a9-89e6-e6f35382ac72"
 					(reference "J2")
@@
 		)
 		(instances
-			(project "keys-lefthand"
+			(project "keys-righthand"
 				(path "/9764b4ba-7c88-49a9-89e6-e6f35382ac72"
 					(reference "J3")
@@
 		)
 		(instances
-			(project "keys-lefthand"
+			(project "keys-righthand"
 				(path "/9764b4ba-7c88-49a9-89e6-e6f35382ac72"
 					(page "2")
@@
 		)
 		(instances
-			(project "keys-lefthand"
+			(project "keys-righthand"
 				(path "/9764b4ba-7c88-49a9-89e6-e6f35382ac72"
 					(page "3")
