File: keys-lefthand/keys-lefthand.kicad_pcb (KiCad board)
At the start: 2 copper layers, 190.5 x 229.6 mm, 83 parts, among them J1 Conn_01x20, J2 Conn_01x20, J3 Conn_01x20, J4 Conn_01x20

Commit message: pcb: Update revision numbers
Signed-off-by: Dylan Turner <dylan.turner@tutanota.com>
Other:
- board text added: "r3"
- board text removed: "r2"
Changed lines of the file:
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@@
 	(title_block
 		(title "PS-OHK")
-		(date "2024-06-18")
-		(rev "2")
+		(date "2024-06-25")
+		(rev "3")
 		(company "Polymath-Studio")
 	)
@@
 		)
 	)
-	(gr_text "r2"
+	(gr_text "r3"
 		(at 69.596 44.704 0)
 		(layer "B.SilkS")

Commit message: r4: 1mm->2.54mm pins, no right-hand yet
Signed-off-by: Dylan Turner <dylan.turner@tutanota.com>
Parts:
- J1, J2, J3, J4: footprint Connector_PinHeader_1.00mm:PinHeader_1x20_P1.00mm_Vertical -> Connector_PinHeader_2.54mm:PinHeader_1x20_P2.54mm_Vertical
- moved J1 66.3 mm to (258.3, 60.5)
- moved J3 45.0 mm to (206.0, 165.5)
- moved J4 39.3 mm to (210.0, 169.5)
- moved J2 35.1 mm to (206.0, 113.0)
Routing:
- net GND: track 1841.2 -> 1931.2 mm, vias 13 -> 16
- net /KEY_BACKSPACE: track 163.3 -> 247.2 mm, vias 3 -> 4
- net /KEY_REAL_6: track 139.8 -> 221.5 mm, vias 2 -> 3
- net /KEY_LEFT: track 242.9 -> 316.1 mm, vias 3 -> 8
- net /KEY_F9: track 113.0 -> 181.0 mm, vias 4 -> 6
- net /KEY_UP: track 211.5 -> 279.1 mm, vias 2 -> 7
- net /KEY_F10: track 116.8 -> 182.3 mm, vias 4 -> 8
- net /KEY_F11: track 69.5 -> 133.7 mm, vias 2 -> 6
- net /KEY_DOWN: track 235.4 -> 297.8 mm, vias 2 -> 6
- net /KEY_RIGHT: track 209.5 -> 271.9 mm, vias 2 -> 4
- net /KEY_K: track 189.6 -> 251.1 mm, vias 3 -> 5
- net /KEY_Y: track 88.0 -> 149.2 mm, vias 3 -> 6
- net /KEY_G: track 153.6 -> 214.4 mm, vias 2 -> 4
- net /KEY_L: track 118.9 -> 179.0 mm, vias 2 -> 4
- net /KEY_E: track 74.1 -> 134.1 mm, vias 1 -> 2
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Other:
- board size 190.5 x 229.6 mm -> 252.8 x 229.6 mm
- board text added: "r4"
- board text removed: "r3"
